File: Hardware/ETH1SBATT12/ETH1SBATT12.kicad_pcb (KiCad board)
At the start: 2 copper layers, 167 x 100 mm, 128 parts, among them J201 20021111-00010T4LF, J301 1715721, J501 RJ45_Wuerth_7499010121A, J601 20021111-00010T4LF, J701 DE9_Receptacle, K401 G5V-2, Q301 SUD09P10-195, Q302 MMBT3904, Q401 MMBT3904, SW601 SW_DIP_x04, U201 RI3-2409S, U202 ISO1044BD, U203 STM32F103T8U7TR, U204 LT1963EQ, U205 MCP1703AT-3302E/MB, U206 INA190AxIDC, U207 OPA376AIDBVR, U208 AD5683R, U209 OPA197xDBV, U301 TSR_1-2433, U302 TSR_1-2450, U501 LAN8742A, U601 STM32H743VITx, U602 24LC08B-E/MS, Y501 NX5032GA-25, Y601 NX5032GA-16

Commit message: Hardware design
Parts:
- added J802: Conn_02x05_Odd_Even, Connector_PinHeader_2.54mm:PinHeader_2x05_P2.54mm_Vertical, F.Cu at (167.5, 124.5)
- moved C202 2.50 mm to (126.5, 131.2)
- moved C203 2.50 mm to (121.4, 140.5)
- moved C205 2.50 mm to (121.4, 131.2)
- moved C206 2.50 mm to (120.8, 128.0)
- moved C207 2.50 mm to (113.4, 142.1)
- moved C209 2.50 mm to (103.3, 128.5)
- moved C211 2.50 mm to (110.2, 142.1)
- moved C212 2.50 mm to (95.2, 129.5)
- moved C215 2.50 mm to (113.7, 123.7)
- moved C217 2.50 mm to (119.3, 133.7)
- moved C219 2.50 mm to (108.3, 124.5)
- moved C223 2.50 mm to (110.7, 127.0)
- moved D201 2.50 mm to (111.4, 137.5)
- moved D202 2.50 mm to (111.4, 138.7)
- moved R201 2.50 mm to (111.4, 137.5)
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