File: Hardware/ETH1SBATT12/ETH1SBATT12.kicad_sch (KiCad schematic)
At the start: 0 parts

Commit message: Hardware design
Other:
- added sheet Module Connector (ModuleConnector.kicad_sch)
Changed lines of the file:
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@@
+	)
+	(sheet
+		(at 93.98 101.6)
+		(size 27.94 27.94)
+		(fields_autoplaced yes)
+		(stroke
+			(width 0.1524)
+			(type solid)
+		)
+		(fill
+			(color 0 0 0 0.0000)
+		)
+		(property "Sheetname" "Module Connector"
+			(at 93.98 100.8884 0)
+			(effects
+				(font
+					(size 1.27 1.27)
+				)
+				(justify left bottom)
+			)
+		)
+		(property "Sheetfile" "ModuleConnector.kicad_sch"
+			(at 93.98 130.1246 0)
+			(effects
+				(font
+					(size 1.27 1.27)
+				)
+				(justify left top)
+			)
+		)
+		(instances
+			(project "ETH1SBATT12"
+				(path "/65cd6103-a85c-466d-b20c-84253dfc9c3b"
+					(page "8")
+				)
+			)
+		)
 	)
 	(sheet
